Commit message: remove <transmission>

File: source/hanu_lab/data/Robots/hanu/LegV5_URDF_Export_description/urdf/LegV5.urdf (robot description, URDF)
Before this commit: robot LegV5_URDF_Export, 17 links, 16 joints
Links:
- link L11_Knee_Pitch_1_1: geometry collision mesh filename=/home/ubuntu/hanu_lab/hanu_lab/source/hanu_lab/data/Robots/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 scale=0.001 0.001 0.001; visual mesh filename=/home/ubuntu/hanu_lab/hanu_lab/source/hanu_lab/data/Robots/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 scale=0.001 0.001 0.001
- link L13_Foot_1_1: geometry collision mesh filename=/home/ubuntu/hanu_lab/hanu_lab/source/hanu_lab/data/Robots/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 scale=0.001 0.001 0.001; visual mesh filename=/home/ubuntu/hanu_lab/hanu_lab/source/hanu_lab/data/Robots/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 scale=0.001 0.001 0.001
- link L1_Hip_1_1: geometry collision mesh filename=/home/ubuntu/hanu_lab/hanu_lab/source/hanu_lab/data/Robots/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 scale=0.001 0.001 0.001; visual mesh filename=/home/ubuntu/hanu_lab/hanu_lab/source/hanu_lab/data/Robots/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 scale=0.001 0.001 0.001
- link L2_Hip_1_1: geometry collision mesh filename=/home/ubuntu/hanu_lab/hanu_lab/source/hanu_lab/data/Robots/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 scale=0.001 0.001 0.001; visual mesh filename=/home/ubuntu/hanu_lab/hanu_lab/source/hanu_lab/data/Robots/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 scale=0.001 0.001 0.001
- link L3_Upper_1_1: geometry collision mesh filename=/home/ubuntu/hanu_lab/hanu_lab/source/hanu_lab/data/Robots/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 scale=0.001 0.001 0.001; visual mesh filename=/home/ubuntu/hanu_lab/hanu_lab/source/hanu_lab/data/Robots/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 scale=0.001 0.001 0.001
- link L4_Lower_1_1: geometry collision mesh filename=/home/ubuntu/hanu_lab/hanu_lab/source/hanu_lab/data/Robots/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 scale=0.001 0.001 0.001; visual mesh filename=/home/ubuntu/hanu_lab/hanu_lab/source/hanu_lab/data/Robots/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 scale=0.001 0.001 0.001
- link L5_Knee_Roll_1_1: geometry collision mesh filename=/home/ubuntu/hanu_lab/hanu_lab/source/hanu_lab/data/Robots/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 scale=0.001 0.001 0.001; visual mesh filename=/home/ubuntu/hanu_lab/hanu_lab/source/hanu_lab/data/Robots/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 scale=0.001 0.001 0.001
- link L6_U_Joint_1_1: geometry collision mesh filename=/home/ubuntu/hanu_lab/hanu_lab/source/hanu_lab/data/Robots/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 scale=0.001 0.001 0.001; visual mesh filename=/home/ubuntu/hanu_lab/hanu_lab/source/hanu_lab/data/Robots/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 scale=0.001 0.001 0.001
- link R11_Knee_Pitch_1_1: geometry collision mesh filename=/home/ubuntu/hanu_lab/hanu_lab/source/hanu_lab/data/Robots/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 scale=0.001 0.001 0.001; visual mesh filename=/home/ubuntu/hanu_lab/hanu_lab/source/hanu_lab/data/Robots/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 scale=0.001 0.001 0.001
- link R13_Foot_1_1: geometry collision mesh filename=/home/ubuntu/hanu_lab/hanu_lab/source/hanu_lab/data/Robots/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 scale=0.001 0.001 0.001; visual mesh filename=/home/ubuntu/hanu_lab/hanu_lab/source/hanu_lab/data/Robots/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 scale=0.001 0.001 0.001
- link R1_Hip_1_1: geometry collision mesh filename=/home/ubuntu/hanu_lab/hanu_lab/source/hanu_lab/data/Robots/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 scale=0.001 0.001 0.001; visual mesh filename=/home/ubuntu/hanu_lab/hanu_lab/source/hanu_lab/data/Robots/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 scale=0.001 0.001 0.001
- link R2_Hip_1_1: geometry collision mesh filename=/home/ubuntu/hanu_lab/hanu_lab/source/hanu_lab/data/Robots/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 scale=0.001 0.001 0.001; visual mesh filename=/home/ubuntu/hanu_lab/hanu_lab/source/hanu_lab/data/Robots/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 scale=0.001 0.001 0.001
- link R3_Upper_1_1: geometry collision mesh filename=/home/ubuntu/hanu_lab/hanu_lab/source/hanu_lab/data/Robots/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 scale=0.001 0.001 0.001; visual mesh filename=/home/ubuntu/hanu_lab/hanu_lab/source/hanu_lab/data/Robots/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 scale=0.001 0.001 0.001
- link R4_Lower_1_1: geometry collision mesh filename=/home/ubuntu/hanu_lab/hanu_lab/source/hanu_lab/data/Robots/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 scale=0.001 0.001 0.001; visual mesh filename=/home/ubuntu/hanu_lab/hanu_lab/source/hanu_lab/data/Robots/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 scale=0.001 0.001 0.001
- link R5_Knee_Roll_1_1: geometry collision mesh filename=/home/ubuntu/hanu_lab/hanu_lab/source/hanu_lab/data/Robots/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 scale=0.001 0.001 0.001; visual mesh filename=/home/ubuntu/hanu_lab/hanu_lab/source/hanu_lab/data/Robots/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 scale=0.001 0.001 0.001
- link R6_U_Joint_1_1: geometry collision mesh filename=/home/ubuntu/hanu_lab/hanu_lab/source/hanu_lab/data/Robots/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 scale=0.001 0.001 0.001; visual mesh filename=/home/ubuntu/hanu_lab/hanu_lab/source/hanu_lab/data/Robots/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 scale=0.001 0.001 0.001
- link base_link: geometry collision mesh filename=/home/ubuntu/hanu_lab/hanu_lab/source/hanu_lab/data/Robots/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 scale=0.001 0.001 0.001; visual mesh filename=/home/ubuntu/hanu_lab/hanu_lab/source/hanu_lab/data/Robots/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 scale=0.001 0.001 0.001
