Commit message: add action_history in ObsCfg

File: source/hanu_lab/data/Robots/hanu/hanu_a4_description/urdf/hanu_a4.urdf (robot description, URDF)
Before this commit: robot hanu_a4, 37 links, 36 joints
Joints:
- joint Joint_E1R: type revolute -> fixed
- joint Joint_l_hip_roll: limit lower=-0.173958 upper=1.570796 effort=72 velocity=2.27 -> lower=0.0 upper=1.570796 effort=72 velocity=2.27
- joint Joint_l_wrist_pitch: type revolute -> fixed
- joint Joint_l_wrist_roll: type revolute -> fixed
- joint Joint_l_wrist_yaw: type revolute -> fixed
- joint Joint_r_hip_roll: limit lower=-0.173958 upper=1.570796 effort=72 velocity=2.27 -> lower=0.0 upper=1.570796 effort=72 velocity=2.27
- joint Joint_r_wrist_pitch: type revolute -> fixed
- joint Joint_r_wrist_roll: type revolute -> fixed
- joint Joint_r_wrist_yaw: type revolute -> fixed

Commit message: add PD tuning for Explicit Actuator

File: source/hanu_lab/data/Robots/hanu/hanu_a4_description/urdf/hanu_a4.urdf (robot description, URDF)
Before this commit: robot hanu_a4, 37 links, 36 joints
Links:
- link E1R_1: geometry collision mesh filename=../meshes/E1R_1.stl scale=0.001 0.001 0.001; visual mesh filename=../meshes/E1R_1.stl scale=0.001 0.001 0.001
- link abdomen_1: geometry collision mesh filename=../meshes/abdomen_1.stl scale=0.001 0.001 0.001; visual mesh filename=../meshes/abdomen_1.stl scale=0.001 0.001 0.001
- link base_link: geometry collision mesh filename=../meshes/base_link.stl scale=0.001 0.001 0.001; visual mesh filename=../meshes/base_link.stl scale=0.001 0.001 0.001
- link fixed_imu_1: geometry collision mesh filename=../meshes/fixed_imu_1.stl scale=0.001 0.001 0.001; visual mesh filename=../meshes/fixed_imu_1.stl scale=0.001 0.001 0.001
- link fixed_mid_360_1: geometry collision mesh filename=../meshes/fixed_mid_360_1.stl scale=0.001 0.001 0.001; visual mesh filename=../meshes/fixed_mid_360_1.stl scale=0.001 0.001 0.001
- link head_1: geometry collision mesh filename=../meshes/head_1.stl scale=0.001 0.001 0.001; visual mesh filename=../meshes/head_1.stl scale=0.001 0.001 0.001
- link l_ankle_pitch_1: geometry collision mesh filename=../meshes/l_ankle_pitch_1.stl scale=0.001 0.001 0.001; visual mesh filename=../meshes/l_ankle_pitch_1.stl scale=0.001 0.001 0.001
- link l_calf_pitch_1: geometry collision mesh filename=../meshes/l_calf_pitch_1.stl scale=0.001 0.001 0.001; visual mesh filename=../meshes/l_calf_pitch_1.stl scale=0.001 0.001 0.001
- link l_contact_sensor_1: geometry collision mesh filename=../meshes/l_contact_sensor_1.stl scale=0.001 0.001 0.001; visual mesh filename=../meshes/l_contact_sensor_1.stl scale=0.001 0.001 0.001
- link l_foot_pressure_sensor_1: geometry collision mesh filename=../meshes/l_foot_pressure_sensor_1.stl scale=0.001 0.001 0.001; visual mesh filename=../meshes/l_foot_pressure_sensor_1.stl scale=0.001 0.001 0.001
- link l_foot_roll_1: geometry collision mesh filename=../meshes/l_foot_roll_1.stl scale=0.001 0.001 0.001; visual mesh filename=../meshes/l_foot_roll_1.stl scale=0.001 0.001 0.001
- link l_glute_pitch_1: geometry collision mesh filename=../meshes/l_glute_pitch_1.stl scale=0.001 0.001 0.001; visual mesh filename=../meshes/l_glute_pitch_1.stl scale=0.001 0.001 0.001
- link l_groin_yaw_1: geometry collision mesh filename=../meshes/l_groin_yaw_1.stl scale=0.001 0.001 0.001; visual mesh filename=../meshes/l_groin_yaw_1.stl scale=0.001 0.001 0.001
- link l_hand_roll_1: geometry collision mesh filename=../meshes/l_hand_roll_1.stl scale=0.001 0.001 0.001; visual mesh filename=../meshes/l_hand_roll_1.stl scale=0.001 0.001 0.001
- link l_lowerarm_pitch_1: geometry collision mesh filename=../meshes/l_lowerarm_pitch_1.stl scale=0.001 0.001 0.001; visual mesh filename=../meshes/l_lowerarm_pitch_1.stl scale=0.001 0.001 0.001
- link l_shoulder_pitch_1: geometry collision mesh filename=../meshes/l_shoulder_pitch_1.stl scale=0.001 0.001 0.001; visual mesh filename=../meshes/l_shoulder_pitch_1.stl scale=0.001 0.001 0.001
- link l_shoulder_roll_1: geometry collision mesh filename=../meshes/l_shoulder_roll_1.stl scale=0.001 0.001 0.001; visual mesh filename=../meshes/l_shoulder_roll_1.stl scale=0.001 0.001 0.001
- link l_thigh_roll_1: geometry collision mesh filename=../meshes/l_thigh_roll_1.stl scale=0.001 0.001 0.001; visual mesh filename=../meshes/l_thigh_roll_1.stl scale=0.001 0.001 0.001
- link l_upperarm_yaw_1: geometry collision mesh filename=../meshes/l_upperarm_yaw_1.stl scale=0.001 0.001 0.001; visual mesh filename=../meshes/l_upperarm_yaw_1.stl scale=0.001 0.001 0.001
- link l_wrist_pitch_1: geometry collision mesh filename=../meshes/l_wrist_pitch_1.stl scale=0.001 0.001 0.001; visual mesh filename=../meshes/l_wrist_pitch_1.stl scale=0.001 0.001 0.001
- link l_wrist_yaw_1: geometry collision mesh filename=../meshes/l_wrist_yaw_1.stl scale=0.001 0.001 0.001; visual mesh filename=../meshes/l_wrist_yaw_1.stl scale=0.001 0.001 0.001
- link neck_1: geometry collision mesh filename=../meshes/neck_1.stl scale=0.001 0.001 0.001; visual mesh filename=../meshes/neck_1.stl scale=0.001 0.001 0.001
- link r_ankle_pitch_1: geometry collision mesh filename=../meshes/r_ankle_pitch_1.stl scale=0.001 0.001 0.001; visual mesh filename=../meshes/r_ankle_pitch_1.stl scale=0.001 0.001 0.001
- link r_calf_pitch_1: geometry collision mesh filename=../meshes/r_calf_pitch_1.stl scale=0.001 0.001 0.001; visual mesh filename=../meshes/r_calf_pitch_1.stl scale=0.001 0.001 0.001
- link r_contact_sensor_1: geometry collision mesh filename=../meshes/r_contact_sensor_1.stl scale=0.001 0.001 0.001; visual mesh filename=../meshes/r_contact_sensor_1.stl scale=0.001 0.001 0.001
- link r_foot_pressure_sensor_1: geometry collision mesh filename=../meshes/r_foot_pressure_sensor_1.stl scale=0.001 0.001 0.001; visual mesh filename=../meshes/r_foot_pressure_sensor_1.stl scale=0.001 0.001 0.001
- link r_foot_roll_1: geometry collision mesh filename=../meshes/r_foot_roll_1.stl scale=0.001 0.001 0.001; visual mesh filename=../meshes/r_foot_roll_1.stl scale=0.001 0.001 0.001
- link r_glute_pitch_1: geometry collision mesh filename=../meshes/r_glute_pitch_1.stl scale=0.001 0.001 0.001; visual mesh filename=../meshes/r_glute_pitch_1.stl scale=0.001 0.001 0.001
- link r_groin_yaw_1: geometry collision mesh filename=../meshes/r_groin_yaw_1.stl scale=0.001 0.001 0.001; visual mesh filename=../meshes/r_groin_yaw_1.stl scale=0.001 0.001 0.001
- link r_hand_roll_1: geometry collision mesh filename=../meshes/r_hand_roll_1.stl scale=0.001 0.001 0.001; visual mesh filename=../meshes/r_hand_roll_1.stl scale=0.001 0.001 0.001
- link r_lowerarm_pitch_1: geometry collision mesh filename=../meshes/r_lowerarm_pitch_1.stl scale=0.001 0.001 0.001; visual mesh filename=../meshes/r_lowerarm_pitch_1.stl scale=0.001 0.001 0.001
- link r_shoulder_pitch_1: geometry collision mesh filename=../meshes/r_shoulder_pitch_1.stl scale=0.001 0.001 0.001; visual mesh filename=../meshes/r_shoulder_pitch_1.stl scale=0.001 0.001 0.001
- link r_shoulder_roll_1: geometry collision mesh filename=../meshes/r_shoulder_roll_1.stl scale=0.001 0.001 0.001; visual mesh filename=../meshes/r_shoulder_roll_1.stl scale=0.001 0.001 0.001
- link r_thigh_roll_1: geometry collision mesh filename=../meshes/r_thigh_roll_1.stl scale=0.001 0.001 0.001; visual mesh filename=../meshes/r_thigh_roll_1.stl scale=0.001 0.001 0.001
- link r_upperarm_yaw_1: geometry collision mesh filename=../meshes/r_upperarm_yaw_1.stl scale=0.001 0.001 0.001; visual mesh filename=../meshes/r_upperarm_yaw_1.stl scale=0.001 0.001 0.001
- link r_wrist_pitch_1: geometry collision mesh filename=../meshes/r_wrist_pitch_1.stl scale=0.001 0.001 0.001; visual mesh filename=../meshes/r_wrist_pitch_1.stl scale=0.001 0.001 0.001
- link r_wrist_yaw_1: geometry collision mesh filename=../meshes/r_wrist_yaw_1.stl scale=0.001 0.001 0.001; visual mesh filename=../meshes/r_wrist_yaw_1.stl scale=0.001 0.001 0.001
